File: hardware/LogicGates/nand.brd (EAGLE design)
At the start: 36 x 30 mm, 13 parts

Commit message: adding logo
Parts:
- added U$1: CMD_C0DE_LOGOCMD_CODE_LOGO_TOP_COPPER, logos:CMD_C0DE_LOGO_TOP_COPPER
Changed lines of the file:
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@@
 <attribute name="VALUE" x="-0.635" y="6.35" size="1.27" layer="27" rot="R270"/>
 </element>
+<element name="U$1" library="logos" package="CMD_C0DE_LOGO_TOP_COPPER" value="CMD_C0DE_LOGOCMD_CODE_LOGO_TOP_COPPER" x="31.115" y="26.289" smashed="yes"/>
 </elements>
 <signals>
@@
 <vertex x="0" y="30.48"/>
 <vertex x="0" y="0"/>
-<vertex x="35.56" y="0"/>
-<vertex x="35.56" y="29.21"/>
-<vertex x="34.29" y="30.48"/>
+<vertex x="36.83" y="0"/>
+<vertex x="36.83" y="30.48"/>
 </polygon>
 </signal>

Commit message: made truth table a device
Parts:
- added U$2: NAND_TRUTH_TABLE, logic-gates:NAND_TRUTH_TABLE
Other:
- board text removed: "NAND A B C 0 0 1 0 1 1 1 0 1 1 1 0"
Changed lines of the file:
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@@
 <wire x1="36" y1="30" x2="0" y2="30" width="0" layer="20"/>
 <wire x1="0" y1="30" x2="0" y2="0" width="0" layer="20"/>
-<text x="11.43" y="20" size="1.016" layer="1" font="vector" ratio="16" distance="70">         NAND
-A          B          C
-0          0          1
-0          1          1
-1          0          1
-1          1          0</text>
 <text x="1.27" y="20" size="1.016" layer="1" font="vector">INPUT A</text>
 <text x="29.21" y="20" size="1.016" layer="1" font="vector">INPUT B</text>
@@
 </element>
 <element name="U$1" library="logos" package="CMD_C0DE_LOGO_TOP_COPPER" value="CMD_C0DE_LOGOCMD_CODE_LOGO_TOP_COPPER" x="31.115" y="26.289" smashed="yes"/>
+<element name="U$2" library="logic-gates" package="NAND_TRUTH_TABLE" value="NAND_TRUTH_TABLE" x="11.684" y="19.812" smashed="yes"/>
 </elements>
 <signals>
