File: hardware/LogicGates/nand.brd (EAGLE design)
At the start: 36 x 30 mm, 15 parts

Commit message: make it bigger
Parts:
- removed U$2: NAND_TRUTH_TABLE, logic-gates:NAND_TRUTH_TABLE
- moved U$1 12.0 mm to (37.5, 36.4)
- moved B 2.54 mm to (33.0, 11.4)
- moved R3 1.53 mm to (29.0, 13.8)
- moved PTYPE-2 1.27 mm to (21.6, 15.2)
- moved C2 1.02 mm to (25.8, 11.8)
Routing:
- net VDD: track 73.0 -> 81.2 mm
- net N$3: track 68.2 -> 73.8 mm
- net N$7: track 3.12 -> 4.08 mm
Other:
- board size 36 x 30 mm -> 42 x 40 mm
- board text added: "NAND A B C 0 0 1 0 1 1 1 0 1 1 1 0"
