File: hardware/LogicGates/nand.sch (EAGLE design)
At the start: 13 parts

Commit message: adding logo
Parts:
- added U$1: CMD_C0DE_LOGOCMD_CODE_LOGO_TOP_COPPER, logos:CMD_C0DE_LOGOCMD_CODE_LOGO_TOP_COPPER
Changed lines of the file:
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@@
 <part name="C2" library="passives" deviceset="C-US" device="C1206" value="1 uF"/>
 <part name="J1" library="connector" deviceset="M02" device="1X02_NO_SILK"/>
+<part name="U$1" library="logos" deviceset="CMD_C0DE_LOGO" device="CMD_CODE_LOGO_TOP_COPPER"/>
 </parts>
 <sheets>
@@
 <attribute name="NAME" x="-27.94" y="104.902" size="1.778" layer="95"/>
 </instance>
+<instance part="U$1" gate="G$1" x="88.9" y="55.88" smashed="yes"/>
 </instances>
 <busses>

Commit message: made truth table a device
Parts:
- added U$2: NAND_TRUTH_TABLE, logic-gates:NAND_TRUTH_TABLE
Changed lines of the file:
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@@
 <part name="J1" library="connector" deviceset="M02" device="1X02_NO_SILK"/>
 <part name="U$1" library="logos" deviceset="CMD_C0DE_LOGO" device="CMD_CODE_LOGO_TOP_COPPER"/>
+<part name="U$2" library="logic-gates" deviceset="NAND_TRUTH_TABLE" device=""/>
 </parts>
 <sheets>
@@
 </instance>
 <instance part="U$1" gate="G$1" x="88.9" y="55.88" smashed="yes"/>
+<instance part="U$2" gate="G$1" x="-17.78" y="40.64" smashed="yes"/>
 </instances>
 <busses>
@@
 </schematic>
 </drawing>
+<compatibility>
+<note version="6.3" minversion="6.2.2" severity="warning">
+Since Version 6.2.2 text objects can contain more than one line,
+which will not be processed correctly with this version.
+</note>
+</compatibility>
 </eagle>

Commit message: make it bigger
Parts:
- removed U$2: NAND_TRUTH_TABLE, logic-gates:NAND_TRUTH_TABLE
Changed lines of the file:
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@@
 <part name="J1" library="connector" deviceset="M02" device="1X02_NO_SILK"/>
 <part name="U$1" library="logos" deviceset="CMD_C0DE_LOGO" device="CMD_CODE_LOGO_TOP_COPPER"/>
-<part name="U$2" library="logic-gates" deviceset="NAND_TRUTH_TABLE" device=""/>
 </parts>
 <sheets>
@@
 </instance>
 <instance part="U$1" gate="G$1" x="88.9" y="55.88" smashed="yes"/>
-<instance part="U$2" gate="G$1" x="-17.78" y="40.64" smashed="yes"/>
 </instances>
 <busses>
@@
 </schematic>
 </drawing>
-<compatibility>
-<note version="6.3" minversion="6.2.2" severity="warning">
-Since Version 6.2.2 text objects can contain more than one line,
-which will not be processed correctly with this version.
-</note>
-</compatibility>
 </eagle>
